Commit message: edited robot descriptio to fit real robot

File: description/gazebo_control.xacro (robot description, xacro)
@@ -6,8 +6,8 @@
         <left_joint>left_wheel_joint</left_joint>
         <right_joint>right_wheel_joint</right_joint>
-        <wheel_separation>0.35</wheel_separation>
-        <wheel_diameter>0.1</wheel_diameter>
+        <wheel_separation>0.142</wheel_separation>
+        <wheel_diameter>0.44</wheel_diameter>
         <!--limits-->
-        <max_wheel_torque>100</max_wheel_torque>
+        <max_wheel_torque>50</max_wheel_torque>
         <max_wheel_acceleration>1.0</max_wheel_acceleration>
         <!--output-->

File: description/lidar.xacro (robot description, xacro)
@@ -4,10 +4,10 @@
         <parent link="chassis"/>
         <child link="laser_frame"/>
-        <origin xyz="0.1 0 0.175" rpy="0 0 0"/>
+        <origin xyz="0.1 0 0.1" rpy="0 0 0"/>
     </joint>
     <link name="laser_frame">
         <visual>
             <geometry>
-                <cylinder radius="0.05" length="0.04"/>
+                <cylinder radius="0.035" length="0.02"/>
             </geometry>
             <material name="red"/>
@@ -15,8 +15,8 @@
         <collision>
             <geometry>
-                <cylinder radius="0.05" length="0.04"/>
+                <cylinder radius="0.035" length="0.02"/>
             </geometry>
         </collision>
-        <xacro:inertial_cylinder mass="0.1" length="0.04" radius="0.05">
+        <xacro:inertial_cylinder mass="0.1" radius="0.035" length="0.02">
             <origin xyz="0 0 0" rpy="0 0 0"/>
         </xacro:inertial_cylinder>

File: description/robot.urdf.xacro (robot description, xacro)
@@ -6,4 +6,4 @@
     <xacro:include filename= "lidar.xacro"/> <!--lidar-->
     <!--<xacro:include filename= "camera.xacro"/> -->
-    <xacro:include filename= "depth_camera.xacro"/>
+    <!-- <xacro:include filename= "depth_camera.xacro"/> -->
 </robot>

File: description/robot_core.xacro (robot description, xacro)
@@ -33,7 +33,7 @@
 <link name="chassis">
     <visual>
-        <origin  xyz="0.15 0 0.075"/>
+        <origin  xyz="0.145 0 0.035"/>
         <geometry>
-            <box size="0.3 0.3 0.15"/>
+            <box size="0.18 0.18 0.07"/>
         </geometry>
         <material name="white">
@@ -41,7 +41,7 @@
     </visual>
     <collision>
-        <origin  xyz="0.15 0 0.075"/>
+        <origin  xyz="0.145 0 0.035"/>
         <geometry>
-            <box size="0.3 0.3 0.15"/>
+            <box size="0.18 0.18 0.07"/>
         </geometry>
     </collision>
@@ -53,9 +53,9 @@
     <material>Gazebo/White</material>
 </gazebo>
-<!-- LEFT WHEEL LINK-->
+<!-- LEFT WHEEL LINK -->
 <joint name="left_wheel_joint" type="continuous">
     <parent link="base_link"/>
     <child link="left_wheel"/>
-    <origin xyz=" 0 0.175 0.0" rpy="-${pi/2} 0.0 0.0"/>
+    <origin xyz=" 0 0.07 0.007" rpy="-${pi/2} 0.0 0.0"/>
     <axis xyz="0.0 0.0 1"/>
 </joint>
@@ -63,5 +63,5 @@
     <visual>
         <geometry>
-            <cylinder radius="0.05" length="0.04"/>
+            <cylinder radius="0.022" length="0.018"/>
         </geometry>
         <material name="blue"/>
@@ -69,8 +69,8 @@
     <collision>
         <geometry>
-            <cylinder radius="0.05" length="0.04"/>
+            <cylinder radius="0.022" length="0.018"/>
         </geometry>
     </collision>
-    <xacro:inertial_cylinder mass="0.1" radius="0.05" length="0.04">
+    <xacro:inertial_cylinder mass="0.02" radius="0.022" length="0.018">
         <origin xyz="0.0 0.0 0.0" rpy="0.0 0.0 0.0"/>
     </xacro:inertial_cylinder>
@@ -83,11 +83,11 @@
     <parent link="base_link"/>
     <child link="right_wheel"/>
-    <origin xyz=" 0 -0.175 0.0" rpy="${pi/2} 0.0 0.0"/>
-    <axis xyz="0.0 0.0 -1"/>
+    <origin xyz=" 0 -0.07 0.007" rpy="${pi/2} 0.0 0.0"/>
+    <axis xyz="0.0 0.0 1"/>
 </joint>
 <link name="right_wheel">
     <visual>
         <geometry>
-            <cylinder radius="0.05" length="0.04"/>
+            <cylinder radius="0.022" length="0.018"/>
         </geometry>
         <material name="blue"/>
@@ -95,8 +95,8 @@
     <collision>
         <geometry>
-            <cylinder radius="0.05" length="0.04"/>
+            <cylinder radius="0.022" length="0.018"/>
         </geometry>
     </collision>
-    <xacro:inertial_cylinder mass="0.1" radius="0.05" length="0.04">
+    <xacro:inertial_cylinder mass="0.02" radius="0.022" length="0.018">
         <origin xyz="0.0 0.0 0.0" rpy="0.0 0.0 0.0"/>
     </xacro:inertial_cylinder>
@@ -109,10 +109,10 @@
     <parent link="chassis"/>
     <child link="caster_wheel"/>
-    <origin xyz="0.24 0 0"/>
+    <origin xyz="0.2 0 0"/>
 </joint>
 <link name="caster_wheel">
     <visual>
         <geometry>
-            <sphere radius="0.05"/>
+            <sphere radius="0.015"/>
         </geometry>
         <material name="green"/>
@@ -120,8 +120,8 @@
     <collision>
         <geometry>
-            <sphere radius="0.05"/>
+            <sphere radius="0.015"/>
         </geometry>
     </collision>
-    <xacro:inertial_sphere mass="0.1" radius="0.05">
+    <xacro:inertial_sphere mass="0.02" radius="0.05">
         <origin xyz="0.0 0.0 0.0" rpy="0.0 0.0 0.0"/>
     </xacro:inertial_sphere>

File: description/ros2_control.xacro (robot description, xacro)
@@ -7,8 +7,8 @@
             <param name="right_wheel_name">right_wheel_joint</param>
             <param name="loop_rate">30</param>
-            <param name="device">/dev/ttyACM0</param>
+            <param name="device">/dev/serial/by-path/platform-fd500000.pcie-pci-0000:01:00.0-usb-0:1.4:1.0</param>
             <param name="baud_rate">57600</param>
             <param name="timeout">1000</param>
-            <param name="enc_counts_per_rev">3436</param>
+            <param name="enc_counts_per_rev">1429</param>
         </hardware>
         <joint name="left_wheel_joint">
