Commit message: fixed typo, updated readme

File: description/lidar.xacro (robot description, xacro)
@@ -19,5 +19,5 @@
         </collision>
         <xacro:inertial_cylinder mass="0.1" radius="0.035" length="0.02">
-            <origin xyz="0 0 0" rpy="0 0 0"/>
+            <origin xyz="0 0 0" rpy="0 0 -${pi/2}"/>
         </xacro:inertial_cylinder>
     </link>
@@ -31,5 +31,5 @@
                 <scan>
                     <horizontal>
-                        <samples>360</samples>
+                        <samples>720</samples>
                         <min_angle>-3.14</min_angle>
                         <max_angle>3.14</max_angle>

Commit message: fixed wheel spinning and lidar orientation

File: description/lidar.xacro (robot description, xacro)
@@ -4,5 +4,5 @@
         <parent link="chassis"/>
         <child link="laser_frame"/>
-        <origin xyz="0.1 0 0.1" rpy="0 0 0"/>
+        <origin xyz="0.2 0 0.1" rpy="0 0 ${pi/2}"/>
     </joint>
     <link name="laser_frame">
@@ -10,4 +10,5 @@
             <geometry>
                 <cylinder radius="0.035" length="0.02"/>
+                <origin xyz="0 0 0" rpy="0 0 0"/>
             </geometry>
             <material name="red"/>
@@ -19,5 +20,5 @@
         </collision>
         <xacro:inertial_cylinder mass="0.1" radius="0.035" length="0.02">
-            <origin xyz="0 0 0" rpy="0 0 -${pi/2}"/>
+            <origin xyz="0 0 0" rpy="0 0 0"/>
         </xacro:inertial_cylinder>
     </link>
@@ -31,5 +32,5 @@
                 <scan>
                     <horizontal>
-                        <samples>720</samples>
+                        <samples>360</samples>
                         <min_angle>-3.14</min_angle>
                         <max_angle>3.14</max_angle>

File: description/robot_core.xacro (robot description, xacro)
@@ -83,5 +83,5 @@
     <parent link="base_link"/>
     <child link="right_wheel"/>
-    <origin xyz=" 0 -0.07 0.007" rpy="${pi/2} 0.0 0.0"/>
+    <origin xyz=" 0 -0.07 0.007" rpy="-${pi/2} 0.0 0.0"/>
     <axis xyz="0.0 0.0 1"/>
 </joint>
