Commit message: Update Readme fixed robot description

File: description/robot.urdf.xacro (robot description, xacro)
@@ -1,5 +1,5 @@
 <?xml version="1.0"?>
 <robot xmlns:xacro="http://www.ros.org/wiki/xacro"  name="robot">
-    <xacro:include filename= "robot_core_big_wheels.xacro"/> <!--Base model of robo and wheels-->
+    <xacro:include filename= "robot_core.xacro"/> <!--Base model of robo and wheels-->
     <!-- <xacro:include filename= "gazebo_control.xacro"/> Parameters for simulating in Gazebo -->
     <xacro:include filename= "ros2_control_real.xacro"/> <!--Parameters for simulating in Gazebo-->

File: description/robot_core.xacro (robot description, xacro)
@@ -29,5 +29,5 @@
     <parent link="base_link"/>
     <child link="chassis"/>
-    <origin xyz= "-0.1 0 0"/>
+    <origin xyz= "-0.07 0 0"/>
 </joint>
 <link name="chassis">
@@ -57,5 +57,5 @@
     <parent link="base_link"/>
     <child link="left_wheel"/>
-    <origin xyz=" 0 0.07 0.007" rpy="-${pi/2} 0.0 0.0"/>
+    <origin xyz=" 0 0.1 0.00" rpy="-${pi/2} 0.0 0.0"/>
     <axis xyz="0.0 0.0 1"/>
 </joint>
@@ -63,5 +63,5 @@
     <visual>
         <geometry>
-            <cylinder radius="0.022" length="0.018"/>
+            <cylinder radius="0.03" length="0.01"/>
         </geometry>
         <material name="blue"/>
@@ -69,8 +69,8 @@
     <collision>
         <geometry>
-            <cylinder radius="0.022" length="0.018"/>
+            <cylinder radius="0.03" length="0.01"/>
         </geometry>
     </collision>
-    <xacro:inertial_cylinder mass="0.02" radius="0.022" length="0.018">
+    <xacro:inertial_cylinder mass="0.02" radius="0.03" length="0.01">
         <origin xyz="0.0 0.0 0.0" rpy="0.0 0.0 0.0"/>
     </xacro:inertial_cylinder>
@@ -83,5 +83,5 @@
     <parent link="base_link"/>
     <child link="right_wheel"/>
-    <origin xyz=" 0 -0.07 0.007" rpy="-${pi/2} 0.0 0.0"/>
+    <origin xyz=" 0 -0.1 0.00" rpy="-${pi/2} 0.0 0.0"/>
     <axis xyz="0.0 0.0 1"/>
 </joint>
@@ -89,5 +89,5 @@
     <visual>
         <geometry>
-            <cylinder radius="0.022" length="0.018"/>
+            <cylinder radius="0.03" length="0.01"/>
         </geometry>
         <material name="blue"/>
@@ -95,8 +95,8 @@
     <collision>
         <geometry>
-            <cylinder radius="0.022" length="0.018"/>
+            <cylinder radius="0.03" length="0.01"/>
         </geometry>
     </collision>
-    <xacro:inertial_cylinder mass="0.02" radius="0.022" length="0.018">
+    <xacro:inertial_cylinder mass="0.02" radius="0.03" length="0.01">
         <origin xyz="0.0 0.0 0.0" rpy="0.0 0.0 0.0"/>
     </xacro:inertial_cylinder>
@@ -114,5 +114,5 @@
     <visual>
         <geometry>
-            <sphere radius="0.015"/>
+            <sphere radius="0.03"/>
         </geometry>
         <material name="green"/>
@@ -120,8 +120,8 @@
     <collision>
         <geometry>
-            <sphere radius="0.015"/>
+            <sphere radius="0.03"/>
         </geometry>
     </collision>
-    <xacro:inertial_sphere mass="0.02" radius="0.05">
+    <xacro:inertial_sphere mass="0.02" radius="0.03">
         <origin xyz="0.0 0.0 0.0" rpy="0.0 0.0 0.0"/>
     </xacro:inertial_sphere>

File: description/robot_core_old.xacro (robot description, xacro)
@@ -29,5 +29,5 @@
     <parent link="base_link"/>
     <child link="chassis"/>
-    <origin xyz= "-0.07 0 0"/>
+    <origin xyz= "-0.1 0 0"/>
 </joint>
 <link name="chassis">
@@ -57,5 +57,5 @@
     <parent link="base_link"/>
     <child link="left_wheel"/>
-    <origin xyz=" 0 0.1 0.00" rpy="-${pi/2} 0.0 0.0"/>
+    <origin xyz=" 0 0.07 0.007" rpy="-${pi/2} 0.0 0.0"/>
     <axis xyz="0.0 0.0 1"/>
 </joint>
@@ -63,5 +63,5 @@
     <visual>
         <geometry>
-            <cylinder radius="0.03" length="0.01"/>
+            <cylinder radius="0.022" length="0.018"/>
         </geometry>
         <material name="blue"/>
@@ -69,8 +69,8 @@
     <collision>
         <geometry>
-            <cylinder radius="0.03" length="0.01"/>
+            <cylinder radius="0.022" length="0.018"/>
         </geometry>
     </collision>
-    <xacro:inertial_cylinder mass="0.02" radius="0.03" length="0.01">
+    <xacro:inertial_cylinder mass="0.02" radius="0.022" length="0.018">
         <origin xyz="0.0 0.0 0.0" rpy="0.0 0.0 0.0"/>
     </xacro:inertial_cylinder>
@@ -83,5 +83,5 @@
     <parent link="base_link"/>
     <child link="right_wheel"/>
-    <origin xyz=" 0 -0.1 0.00" rpy="-${pi/2} 0.0 0.0"/>
+    <origin xyz=" 0 -0.07 0.007" rpy="-${pi/2} 0.0 0.0"/>
     <axis xyz="0.0 0.0 1"/>
 </joint>
@@ -89,5 +89,5 @@
     <visual>
         <geometry>
-            <cylinder radius="0.03" length="0.01"/>
+            <cylinder radius="0.022" length="0.018"/>
         </geometry>
         <material name="blue"/>
@@ -95,8 +95,8 @@
     <collision>
         <geometry>
-            <cylinder radius="0.03" length="0.01"/>
+            <cylinder radius="0.022" length="0.018"/>
         </geometry>
     </collision>
-    <xacro:inertial_cylinder mass="0.02" radius="0.03" length="0.01">
+    <xacro:inertial_cylinder mass="0.02" radius="0.022" length="0.018">
         <origin xyz="0.0 0.0 0.0" rpy="0.0 0.0 0.0"/>
     </xacro:inertial_cylinder>
@@ -114,5 +114,5 @@
     <visual>
         <geometry>
-            <sphere radius="0.03"/>
+            <sphere radius="0.015"/>
         </geometry>
         <material name="green"/>
@@ -120,8 +120,8 @@
     <collision>
         <geometry>
-            <sphere radius="0.03"/>
+            <sphere radius="0.015"/>
         </geometry>
     </collision>
-    <xacro:inertial_sphere mass="0.02" radius="0.03">
+    <xacro:inertial_sphere mass="0.02" radius="0.05">
         <origin xyz="0.0 0.0 0.0" rpy="0.0 0.0 0.0"/>
     </xacro:inertial_sphere>

Commit message: sorted out operation modes

File: description/robot.urdf.xacro (robot description, xacro)
@@ -2,7 +2,7 @@
 <robot xmlns:xacro="http://www.ros.org/wiki/xacro"  name="robot">
     <xacro:include filename= "robot_core.xacro"/> <!--Base model of robo and wheels-->
-    <!-- <xacro:include filename= "gazebo_control.xacro"/> Parameters for simulating in Gazebo -->
-    <xacro:include filename= "ros2_control_real.xacro"/> <!--Parameters for simulating in Gazebo-->
-    <!-- <xacro:include filename= "ros2_control_sim.xacro"/> -->
+    <!--<xacro:include filename= "gazebo_control.xacro"/> Simulation WITHOUT ros2 control-->
+    <xacro:include filename= "ros2_control_real.xacro"/>  <!--Real robot with ros2 control-->
+    <!-- <xacro:include filename= "ros2_control_sim.xacro"/> Simulation WITH ros2 control-->
     <xacro:include filename= "lidar.xacro"/> <!--lidar-->
     <!--<xacro:include filename= "camera.xacro"/> -->

File: description/ros2_control_real.xacro (robot description, xacro)
@@ -29,31 +29,7 @@
         </joint>
     </ros2_control>
-    <!-- <xacro:if value="$(arg sim_mode)">
-        <ros2_control name="GazeboSystem" type="system">
-            <hardware>
-                <plugin>gazebo_ros2_control/GazeboSystem</plugin>
-            </hardware>
-            <joint name="left_wheel_joint">
-                <command_interface name="velocity">
-                    <param name="min">-10</param>
-                    <param name="max">10</param>
-                </command_interface>
-                <state_interface name="velocity"/>
-                <state_interface name="position"/>
-            </joint>
-            <joint name="right_wheel_joint">
-                <command_interface name="velocity">
-                    <param name="min">-10</param>
-                    <param name="max">10</param>
-                </command_interface>
-                <state_interface name="velocity"/>
-                <state_interface name="position"/>
-            </joint>
-        </ros2_control>
-    </xacro:if> -->
     <gazebo>
         <plugin name="gazebo_ros2_control" filename="libgazebo_ros2_control.so">
             <parameters>$(find my_bot)/config/my_controllers.yaml</parameters>
-            <parameters>$(find my_bot)/config/gaz_ros2_ctl_use_sim.yaml</parameters>
         </plugin>
     </gazebo>
