Commit message: modified for new chasis

File: diffdrive_arduino/description/ros2_control/diffbot.ros2_control.xacro (robot description, xacro)
@@ -4,5 +4,5 @@
     <ros2_control name="${name}" type="system">
       <hardware>
-        <plugin>diffdrive_arduino/DiffDriveArduinoHardware</plugin>
+        <!-- <plugin>diffdrive_arduino/DiffDriveArduinoHardware</plugin>
         <param name="left_wheel_name">left_wheel_joint</param>
         <param name="right_wheel_name">right_wheel_joint</param>
@@ -15,7 +15,7 @@
         <param name="pid_d">12</param>
         <param name="pid_i">0</param>
-        <param name="pid_o">50</param>
+        <param name="pid_o">50</param> -->
       </hardware>
-      <joint name="${prefix}left_wheel_joint">
+      <!-- <joint name="${prefix}left_wheel_joint">
         <command_interface name="velocity"/>
         <state_interface name="position"/>
@@ -34,5 +34,5 @@
         <command_interface name="cmd_val"/>
         <state_interface name="cmd_val"/>
-      </gpio>
+      </gpio> -->
     </ros2_control>
   </xacro:macro>

File: diffdrive_arduino/description/urdf/diffbot_description.urdf.xacro (robot description, xacro)
@@ -46,5 +46,5 @@
     </joint>
     <!-- left wheel Link -->
-    <link name="${prefix}left_wheel">
+    <!-- <link name="${prefix}left_wheel">
       <collision>
         <origin xyz="0 0 0" rpy="${PI/2} 0 0"/>
@@ -75,7 +75,7 @@
       <axis xyz="0 1 0"/>
       <dynamics damping="0.2"/>
-    </joint>
+    </joint> -->
     <!-- right wheel Link -->
-    <link name="${prefix}right_wheel">
+    <!-- <link name="${prefix}right_wheel">
       <collision>
         <origin xyz="0 0 0" rpy="${PI/2} 0 0"/>
@@ -104,7 +104,7 @@
       <child link="${prefix}caster_frontal_wheel"/>
       <origin xyz="${base_width/2 - caster_wheel_radius} 0 ${z_offset}" rpy="0 0 0"/>
-    </joint>
+    </joint> -->
     <!-- caster frontal wheel Link -->
-    <link name="${prefix}caster_frontal_wheel">
+    <!-- <link name="${prefix}caster_frontal_wheel">
       <collision>
         <origin xyz="0 0 0" rpy="0 0 0"/>
@@ -133,7 +133,7 @@
       <child link="${prefix}caster_rear_wheel"/>
       <origin xyz="${-base_width/2 + caster_wheel_radius} 0 ${z_offset}" rpy="0 0 0"/>
-    </joint>
+    </joint> -->
     <!-- caster rear wheel Link -->
-    <link name="${prefix}caster_rear_wheel">
+    <!-- <link name="${prefix}caster_rear_wheel">
       <collision>
         <origin xyz="0 0 0" rpy="0 0 0"/>
@@ -157,5 +157,5 @@
           izz="${caster_wheel_mass * 0.4 * (caster_wheel_radius * caster_wheel_radius)}"/>
         </inertial>
-      </link>
+      </link> -->
   </xacro:macro>
 </robot>

File: my_bot/description/robot.urdf.xacro (robot description, xacro)
@@ -3,5 +3,5 @@
     <xacro:include filename= "robot_core.xacro"/> <!--Base model of robo and wheels-->
     <!--<xacro:include filename= "gazebo_control.xacro"/> Simulation WITHOUT ros2 control-->
-    <xacro:include filename= "ros2_control_real.xacro"/>  <!--Real robot with ros2 control-->
+    <xacro:include filename= "ros2_control_real.xacro"/>  <!-- Real robot with ros2 control -->
     <!-- <xacro:include filename= "ros2_control_sim.xacro"/> Simulation WITH ros2 control-->
    <!-- <xacro:include filename= "lidar.xacro"/> lidar-->

File: my_bot/description/robot_core.xacro (robot description, xacro)
@@ -29,11 +29,11 @@
     <parent link="base_link"/>
     <child link="chassis"/>
-    <origin xyz= "-0.07 0 0"/>
+    <origin xyz= "0 0 0"/>
 </joint>
 <link name="chassis">
     <visual>
-        <origin  xyz="0.145 0 0.035"/>
+        <origin  xyz="0.06 0 0.035"/>
         <geometry>
-            <box size="0.18 0.18 0.07"/>
+            <cylinder radius="0.145" length="0.08"/>
         </geometry>
         <material name="white">
@@ -41,7 +41,7 @@
     </visual>
     <collision>
-        <origin  xyz="0.145 0 0.035"/>
+        <origin  xyz="0.06 0 0.035"/>
         <geometry>
-            <box size="0.18 0.18 0.07"/>
+            <cylinder radius="0.145" length="0.08"/>
         </geometry>
     </collision>
@@ -57,5 +57,5 @@
     <parent link="base_link"/>
     <child link="left_wheel"/>
-    <origin xyz=" 0 0.1 0.00" rpy="-${pi/2} 0.0 0.0"/>
+    <origin xyz=" 0 0.09 0.00" rpy="-${pi/2} 0.0 0.0"/>
     <axis xyz="0.0 0.0 1"/>
 </joint>
@@ -63,5 +63,5 @@
     <visual>
         <geometry>
-            <cylinder radius="0.03" length="0.01"/>
+            <cylinder radius="0.035" length="0.026"/>
         </geometry>
         <material name="blue"/>
@@ -69,5 +69,5 @@
     <collision>
         <geometry>
-            <cylinder radius="0.03" length="0.01"/>
+            <cylinder radius="0.035" length="0.026"/>
         </geometry>
     </collision>
@@ -83,5 +83,5 @@
     <parent link="base_link"/>
     <child link="right_wheel"/>
-    <origin xyz=" 0 -0.1 0.00" rpy="-${pi/2} 0.0 0.0"/>
+    <origin xyz=" 0 -0.09 0.00" rpy="-${pi/2} 0.0 0.0"/>
     <axis xyz="0.0 0.0 1"/>
 </joint>
@@ -89,5 +89,5 @@
     <visual>
         <geometry>
-            <cylinder radius="0.03" length="0.01"/>
+            <cylinder radius="0.035" length="0.026"/>
         </geometry>
         <material name="blue"/>
@@ -95,5 +95,5 @@
     <collision>
         <geometry>
-            <cylinder radius="0.03" length="0.01"/>
+            <cylinder radius="0.035" length="0.026"/>
         </geometry>
     </collision>
@@ -109,10 +109,10 @@
     <parent link="chassis"/>
     <child link="caster_wheel"/>
-    <origin xyz="0.2 0 0"/>
+    <origin xyz="0.17 0 -0.015"/>
 </joint>
 <link name="caster_wheel">
     <visual>
         <geometry>
-            <sphere radius="0.03"/>
+            <sphere radius="0.02"/>
         </geometry>
         <material name="green"/>
@@ -120,5 +120,5 @@
     <collision>
         <geometry>
-            <sphere radius="0.03"/>
+            <sphere radius="0.02"/>
         </geometry>
     </collision>
@@ -132,3 +132,30 @@
     <mu2 value="0.001"/>
 </gazebo>
+<!--FRONT MARKER LINK-->
+<joint name="front_marker_joint" type="fixed">
+    <parent link="chassis"/>
+    <child link="front_marker"/>
+    <origin xyz="0.17 0 0.08"/>
+</joint>
+<link name="front_marker">
+    <visual>
+        <geometry>
+            <sphere radius="0.02"/>
+        </geometry>
+        <material name="red"/>
+    </visual>
+    <collision>
+        <geometry>
+            <sphere radius="0.02"/>
+        </geometry>
+    </collision>
+    <xacro:inertial_sphere mass="0.02" radius="0.03">
+        <origin xyz="0.0 0.0 0.0" rpy="0.0 0.0 0.0"/>
+    </xacro:inertial_sphere>
+</link>
+<gazebo reference="front_marker">
+    <material>Gazebo/Red</material>
+    <mu1 value="0.001"/>
+    <mu2 value="0.001"/>
+</gazebo>
 </robot>

File: my_bot/description/ros2_control_real.xacro (robot description, xacro)
@@ -3,5 +3,5 @@
     <ros2_control name="RealRobot" type="system">
         <hardware>
-            <plugin>diffdrive_arduino/DiffDriveArduino</plugin>
+            <plugin>diffdrive_arduino/DiffDriveArduinoHardware</plugin>
             <param name="left_wheel_name">left_wheel_joint</param>
             <param name="right_wheel_name">right_wheel_joint</param>
@@ -10,23 +10,35 @@
             <param name="device">/dev/serial/by-path/pci-0000:02:00.0-usb-0:2.1:1.0-port0</param>
             <param name="baud_rate">57600</param>
-            <param name="timeout">1000</param>
+            <param name="timeout_ms">1000</param>
             <param name="enc_counts_per_rev">10800</param>
+            <param name="pid_p">20</param>
+            <param name="pid_d">12</param>
+            <param name="pid_i">0</param>
+            <param name="pid_o">50</param>
         </hardware>
         <joint name="left_wheel_joint">
-            <command_interface name="velocity">
-                <param name="min">-10</param>
+            <command_interface name="velocity"/>
+                <!-- <param name="min">-10</param>
                 <param name="max">10</param>
-            </command_interface>
+            </command_interface> -->
+            <state_interface name="position"/>
             <state_interface name="velocity"/>
-            <state_interface name="position"/>
         </joint>
         <joint name="right_wheel_joint">
-            <command_interface name="velocity">
-                <param name="min">-10</param>
+            <command_interface name="velocity"/>
+                <!-- <param name="min">-10</param>
                 <param name="max">10</param>
-            </command_interface>
+            </command_interface> -->
+            <state_interface name="position"/>
             <state_interface name="velocity"/>
-            <state_interface name="position"/>
         </joint>
+        <gpio name="test_led1">
+            <command_interface name="cmd_val"/>
+            <state_interface name="cmd_val"/>
+        </gpio>
+        <gpio name="test_led2">
+            <command_interface name="cmd_val"/>
+            <state_interface name="cmd_val"/>
+        </gpio>
     </ros2_control>
     <gazebo>
